Commit message: feat(m3): commit the actual M3/M4 implementation -- was uncommitted since c79dee2
These 14 files were sitting as uncommitted working-tree changes this
entire time: the fingertip-runaway fix (TENTH OVERRIDE -- both fingertip
joints changed from continuous+mimic to fixed in
robotiq_2f_85_macro.urdf.xacro, dropping the mimic count from five to
three), fingertip_grasp_theta threaded through scene_xacro_args.py and
every launch file that builds robot_description, gripper_geometry.py's
theta_for_width()/aperture_m_fixed_tip(), the retry-until-cycles-actually-
run rewrite of scripts/11_m3_cycles.sh, transport.hpp/transport.cpp's
grasp-loss check and marker-file signaling, and scripts/03_validate_merge.sh's
updated joint-count/joint-type checks.

Every M3/M4/M5 result documented in docs/HANDOFF_M3.md and README.md was
measured against this code, live, this session and prior ones -- the
numbers are real. But none of this had ever been committed, so
origin/main did not reproduce those results from a clean clone. Caught by
external review of a repo export against the README's own claims, not
caught internally before pushing docs that asserted PASS. Fixing that gap
is the entire point of this commit: bringing committed history in line
with what was already true of the working tree, not new functional work.

File: ur5e_robotiq_description/urdf/vendor/robotiq_gripper.ros2_control.xacro (robot description, xacro)
@@ -6,10 +6,10 @@
      reinstall). Same reasoning as vendoring robotiq_2f_85_macro.urdf.xacro
      itself: own the file, track the diff.
-     ONE CHANGE from upstream: the actuated joint
+     CHANGE 1 from upstream, 2026-08-11: the actuated joint
      (robotiq_85_left_knuckle_joint) gains a `state_interface name="effort"`.
      gz_system.cpp's read() computes effort from JointTransmittedWrench for
      revolute joints and binds it whenever the interface is declared, so
      this is the only line needed to make it observable on /joint_states.
-     Added 2026-08-11 to test a specific hypothesis: gripper_close_and_hold()
+     Added to test a specific hypothesis: gripper_close_and_hold()
      re-sends its hold at the joint's achieved position rather than the
      original close target (see m3_grasp.cpp), which drives the P-loop's
@@ -18,5 +18,21 @@
      when the lift needs it to hold. This interface turns that from an
      inference (read the code, reason about the control law) into a
-     measurement (read the joint's own effort during the hold). -->
+     measurement (read the joint's own effort during the hold).
+     CHANGE 2 from upstream, 2026-08-12: the actuated joint also gains a
+     `command_interface name="effort"`, alongside (not replacing) the
+     existing position command interface. Confirmed live and derived from
+     the control law: a velocity-servo position controller against a rigid
+     constraint always commands maximum velocity for any non-zero position
+     error, so the commanded value only sets extrusion RATE, never force:
+     it can give bounded extrusion + slack, or sustained force + unbounded
+     extrusion, never sustained force with bounded extrusion, which is what
+     a grasp needs. No effort ceiling on the position interface fixes that;
+     the control law itself is wrong for the hold phase. Position control
+     stays for the close (Stage 2), which reaches touch at 0.4029-0.4038rad
+     across ~60 live cycles, the most reliable behavior in this project,
+     and effort control is for the hold phase only, via a second controller
+     switched in with perform_command_mode_switch. See
+     docs/HANDOFF_M3.md and the pad-force xacro header in
+     robotiq_2f_85_macro.urdf.xacro for the full derivation. -->
 <robot xmlns:xacro="http://www.ros.org/wiki/xacro">
     <xacro:macro name="robotiq_gripper_ros2_control" params="
@@ -56,4 +72,5 @@
             <joint name="${prefix}robotiq_85_left_knuckle_joint">
                 <command_interface name="position" />
+                <command_interface name="effort" />
                 <state_interface name="position">
                     <param name="initial_value">0.7929</param>
@@ -72,4 +89,18 @@
                         <state_interface name="velocity"/>
                     </xacro:unless>
+                    <!-- CHANGE 3 from upstream, 2026-08-12: state-only interfaces added
+                         for sim_ignition too. A mimic-tagged joint cannot carry a
+                         command_interface (ros2_control rejects it), but it can carry
+                         state_interfaces, and without any declared here this joint
+                         never appeared in /joint_states at all (confirmed live: a
+                         2-minute capture against it got 0 rows while the master's
+                         59831). Needed to check HANDOFF_M3.md's "right_knuckle
+                         diverges ~0.027-0.033rad from its multiplier under load"
+                         note directly instead of only through the master's trace. -->
+                    <xacro:if value="${sim_ignition}">
+                        <state_interface name="position"/>
+                        <state_interface name="velocity"/>
+                        <state_interface name="effort"/>
+                    </xacro:if>
                 </joint>
                 <joint name="${prefix}robotiq_85_left_inner_knuckle_joint">
@@ -81,4 +112,15 @@
                         <state_interface name="velocity"/>
                     </xacro:unless>
+                    <!-- CHANGE 3, see right_knuckle_joint above. Added 2026-08-12 to
+                         test the joint_index-1 mimicked-index hypothesis: this is
+                         array index 2 in hardware_info.joints (order:
+                         left_knuckle=0, right_knuckle=1, left_inner_knuckle=2,
+                         right_inner_knuckle=3, left_finger_tip=4,
+                         right_finger_tip=5). -->
+                    <xacro:if value="${sim_ignition}">
+                        <state_interface name="position"/>
+                        <state_interface name="velocity"/>
+                        <state_interface name="effort"/>
+                    </xacro:if>
                 </joint>
                 <joint name="${prefix}robotiq_85_right_inner_knuckle_joint">
@@ -90,23 +132,24 @@
                         <state_interface name="velocity"/>
                     </xacro:unless>
-                </joint>
-                <joint name="${prefix}robotiq_85_left_finger_tip_joint">
-                    <param name="mimic">${prefix}robotiq_85_left_knuckle_joint</param>
-                    <param name="multiplier">-1</param>
-                    <xacro:unless value="${sim_ignition}">
-                        <command_interface name="position"/>
+                    <!-- CHANGE 3, see right_knuckle_joint above. Array index 3. -->
+                    <xacro:if value="${sim_ignition}">
                         <state_interface name="position"/>
                         <state_interface name="velocity"/>
-                    </xacro:unless>
+                        <state_interface name="effort"/>
+                    </xacro:if>
                 </joint>
-                <joint name="${prefix}robotiq_85_right_finger_tip_joint">
-                    <param name="mimic">${prefix}robotiq_85_left_knuckle_joint</param>
-                    <param name="multiplier">1</param>
-                    <xacro:unless value="${sim_ignition}">
-                        <command_interface name="position"/>
-                        <state_interface name="position"/>
-                        <state_interface name="velocity"/>
-                    </xacro:unless>
-                </joint>
+                <!-- CHANGE 5 from upstream, 2026-08-12: left_finger_tip_joint and
+                     right_finger_tip_joint REMOVED from this block entirely.
+                     TENTH OVERRIDE in robotiq_2f_85_macro.urdf.xacro changed both
+                     from continuous+mimic to type="fixed": a fixed joint has
+                     zero DOF and carries no ros2_control interfaces of any kind,
+                     command or state. See that file's TENTH OVERRIDE comment for
+                     the full reasoning (docs/gz_joint_cmd_probe/ traced the
+                     fingertip runaway to dartsim's contact-force resolution
+                     overriding a correctly-computed mimic command; removing the
+                     DOF removes what that resolution had to act on). CHANGE 3/4
+                     above (state interfaces, mimic-reference fix) are dead code
+                     for these two joints now, kept in git history but not
+                     resurrected here. -->
             </xacro:if>
             <!-- Only add this with fake hardware mode -->
