Commit message: style: improve parallel-jaw gripper visualization
Add blue/dark-gray materials to the parallel-jaw gripper's visual
geometry (housing, pads) and add visual-only connector boxes to
jaw_fixed_link/jaw_moving_link, which previously had no <visual>
element at all and left a real, unrendered gap between the housing
and the pads. Visual-only: no collision, joint, inertial, or
controller change.

File: ur5e_robotiq_description/urdf/parallel_jaw_gripper.urdf.xacro (robot description, xacro)
@@ -78,6 +78,9 @@
     - no fingertip_grasp_theta or any object-size-derived xacro argument;
     - visual meshes are NOT attached in this pass (cosmetic vendor-mesh
-      decoration is design §8, not V0 — jaw/base links carry a plain box
-      visual only, so the macro remains self-contained and inspectable).
+      decoration is design §8, not V0 — base/pad links carry a plain box
+      visual, and the two jaw links carry a small visual-only connector box
+      bridging housing to pad (added post-V0, see jaw_fixed_link /
+      jaw_moving_link below), so the macro remains self-contained and
+      inspectable).
   This file must not change the expansion of ur5e_robotiq.urdf.xacro under
   the default gripper_model:=robotiq_linkage in any way, including this
@@ -158,4 +161,7 @@
                     <box size="0.030 0.060 0.030"/>
                 </geometry>
+                <material name="gripper_body_blue">
+                    <color rgba="0.10 0.35 0.90 1.0"/>
+                </material>
             </visual>
             <inertial>
@@ -173,4 +179,17 @@
         <!-- fixed jaw -->
         <link name="${prefix}jaw_fixed_link">
+            <!-- Visual-only connector bridging the housing box to
+                 pad_fixed_link (see this file's audit note above: a real,
+                 unrendered gap otherwise exists between them). No
+                 <collision>: purely cosmetic, does not touch contact/physics. -->
+            <visual>
+                <origin xyz="0.01375 0 -0.022" rpy="0 0 0"/>
+                <geometry>
+                    <box size="0.0315 0.022 0.012"/>
+                </geometry>
+                <material name="gripper_body_blue">
+                    <color rgba="0.10 0.35 0.90 1.0"/>
+                </material>
+            </visual>
             <inertial>
                 <origin xyz="0 0 0" rpy="0 0 0"/>
@@ -190,4 +209,7 @@
                     <box size="${pad_thickness_m} ${pad_width_m} ${pad_height_m}"/>
                 </geometry>
+                <material name="gripper_pad_dark">
+                    <color rgba="0.15 0.15 0.15 1.0"/>
+                </material>
             </visual>
             <collision>
@@ -245,4 +267,18 @@
         <!-- moving jaw — the ONE actuated DOF -->
         <link name="${prefix}jaw_moving_link">
+            <!-- Visual-only connector bridging the housing box to
+                 pad_moving_link, mirrored in X from jaw_fixed_link's
+                 connector. Rides rigidly with this link, so it tracks the
+                 prismatic joint automatically. No <collision>: purely
+                 cosmetic, does not touch contact/physics. -->
+            <visual>
+                <origin xyz="-0.01375 0 -0.022" rpy="0 0 0"/>
+                <geometry>
+                    <box size="0.0315 0.022 0.012"/>
+                </geometry>
+                <material name="gripper_body_blue">
+                    <color rgba="0.10 0.35 0.90 1.0"/>
+                </material>
+            </visual>
             <inertial>
                 <origin xyz="0 0 0" rpy="0 0 0"/>
@@ -268,4 +304,7 @@
                     <box size="${pad_thickness_m} ${pad_width_m} ${pad_height_m}"/>
                 </geometry>
+                <material name="gripper_pad_dark">
+                    <color rgba="0.15 0.15 0.15 1.0"/>
+                </material>
             </visual>
             <collision>

Commit message: fix: correct parallel-jaw pad contact sensor collision references
Both pad contact sensors in parallel_jaw_gripper.urdf.xacro referenced
URDF-side collision names (pad_fixed_link_collision,
pad_moving_link_collision) that do not survive sdformat's fixed-joint
lumping. Verified with `gz sdf -p` on the generated model: the actual
collision names are wrist_3_link_fixed_joint_lump__pad_fixed_link_collision_2
and jaw_moving_link_fixed_joint_lump__pad_moving_link_collision, and neither
old name exists in the converted model. gz::sim::systems::Contact therefore
matched zero collisions and both pad contact streams have been publishing
nothing in every Stage-2A run to date.

Corrected the two <contact><collision> references. Regenerated SDF diff is
exactly those two lines; no link, joint, collision, inertia, friction, or
controller change. Confirmed live 2026-08-29: both contact topics advertise
and both streams captured real contact rows in the Stage-2A O1
configured-center diagnostic control.

File: ur5e_robotiq_description/urdf/parallel_jaw_gripper.urdf.xacro (robot description, xacro)
@@ -257,7 +257,27 @@
                 </surface>
             </collision>
+            <!-- DIAGNOSTIC-ONLY NAME FIX, 2026-08-29. The collision name below
+                 must be the name the collision has AFTER the URDF->SDF
+                 conversion, not the URDF-side name. pad_fixed_link is the
+                 child of a FIXED joint, so sdformat's URDF parser lumps it
+                 into wrist_3_link and renames its collision; it does NOT
+                 rewrite this <contact><collision> reference to match.
+                 Verified with `gz sdf -p` on the generated parallel_jaw URDF:
+                 the model contains
+                   wrist_3_link_fixed_joint_lump__pad_fixed_link_collision_2
+                 and contains NO collision named pad_fixed_link_collision, so
+                 gz::sim::systems::Contact matched nothing and this sensor
+                 published no data at all. That silence is why every Stage-2A
+                 case so far has had to reconstruct pad contact geometrically
+                 instead of measuring it.
+                 The trailing _2 is sdformat's per-link collision counter for
+                 wrist_3_link (wrist_3_link_collision, ..._lump__ur_to_robotiq_link_collision_1,
+                 then this one). If a collision is ever added to or removed
+                 from wrist_3_link, that index moves and this reference goes
+                 silent again, so any run relying on this stream must assert
+                 that contact messages actually arrived, never assume it. -->
             <sensor name="${prefix}pad_fixed_contact" type="contact">
                 <contact>
-                    <collision>${prefix}pad_fixed_link_collision</collision>
+                    <collision>${prefix}wrist_3_link_fixed_joint_lump__${prefix}pad_fixed_link_collision_2</collision>
                 </contact>
                 <update_rate>500</update_rate>
@@ -346,7 +366,13 @@
                 </surface>
             </collision>
+            <!-- DIAGNOSTIC-ONLY NAME FIX, 2026-08-29: same lumping issue as
+                 pad_fixed_contact above. pad_moving_link is lumped into
+                 jaw_moving_link; `gz sdf -p` shows the collision is named
+                 jaw_moving_link_fixed_joint_lump__pad_moving_link_collision
+                 (no numeric suffix, being the only collision on that link).
+                 See the pad_fixed_contact comment for the full rationale. -->
             <sensor name="${prefix}pad_moving_contact" type="contact">
                 <contact>
-                    <collision>${prefix}pad_moving_link_collision</collision>
+                    <collision>${prefix}jaw_moving_link_fixed_joint_lump__${prefix}pad_moving_link_collision</collision>
                 </contact>
                 <update_rate>500</update_rate>

Commit message: feat: add planning-only gripper collision housing

File: ur5e_robotiq_description/urdf/parallel_jaw_gripper.urdf.xacro (robot description, xacro)
@@ -20,11 +20,21 @@
   no closed loop, no protruding collision geometry, no object-dependent
   xacro argument of any kind.
-  KINEMATIC TREE (exactly two collision bodies in the whole gripper):
+  KINEMATIC TREE (exactly two PHYSICAL collision bodies in the whole gripper;
+  see moveit_collision_housing below for the one MoveIt-only planning body):
     parent (gripper_mount_link)
-     └─ (fixed)      gripper_base_link      [NO collision]
+     └─ (fixed)      gripper_base_link      [NO collision, unless
+                                              moveit_collision_housing:=true —
+                                              see that link's own comment]
          ├─ (fixed)      jaw_fixed_link      [NO collision]
          │   └─ (fixed)  pad_fixed_link      [BOX collision + contact sensor]
          └─ (PRISMATIC)  jaw_moving_link     [NO collision]  <- gripper_jaw_joint
              └─ (fixed)  pad_moving_link     [BOX collision + contact sensor]
+  STAGE-3A ADDITION (2026-09-06, design-audited, planning-only): a
+  `moveit_collision_housing` xacro arg, default false, gates ONE additional
+  collision box on gripper_base_link — set true ONLY by move_group's own
+  independent robot_description build, never by the Gazebo/simulation launch,
+  so this changes what MoveIt plans against without changing what Gazebo
+  simulates. See gripper_base_link's own link-level comment for the geometry
+  and its derivation.
   CLOSING AXIS: local +X of gripper_base_link. gripper_jaw_joint's own axis is
   "-1 0 0" (i.e. increasing q moves jaw_moving_link toward -X, toward the
@@ -100,4 +110,5 @@
         fake_sensor_commands:=false
         include_ros2_control:=true
+        moveit_collision_housing:=false
         aperture_m:=0.085
         pad_thickness_m:=0.004
@@ -154,7 +165,24 @@
         <!-- ================================================================= -->
         <link name="${prefix}gripper_base_link">
-            <!-- Visual-only placeholder box. No <collision>: this link must
-                 never be able to touch anything (that is what removes defect 1,
-                 the protruding-collider first-contact problem). -->
+            <!-- Visual-only placeholder box by default (moveit_collision_housing
+                 default false): no <collision>, so this link cannot touch
+                 anything — that is what removes defect 1, the
+                 protruding-collider first-contact problem. When
+                 moveit_collision_housing is true (set ONLY by move_group's own
+                 independent robot_description build, never by the
+                 Gazebo/simulation launch), a single conservative collision box
+                 is added below for MoveIt-side planning/obstacle-awareness
+                 only. Its dimensions are deliberately trimmed from this link's
+                 own 0.030x0.060x0.030 visual box (to 0.020x0.060x0.020) per
+                 the Stage-3A design audit (2026-09-06): the unmodified visual
+                 box was found to leave under 1mm of Z clearance to
+                 PlanningSceneManager's attached pick_target at the validated
+                 30mm-object grasp depth, too thin to certify; the trimmed box
+                 restores a real, derived margin (+2.5mm X / +5.5mm Z) without
+                 touching pad geometry, Gazebo physics, grasp constants, ACM,
+                 or touch_links. jaw_fixed_link/jaw_moving_link deliberately
+                 receive no equivalent geometry — the audit found no
+                 non-degenerate box on either link that stays clear of
+                 pick_target's own volume at that same grasp depth. -->
             <visual>
                 <geometry>
@@ -165,4 +193,12 @@
                 </material>
             </visual>
+            <xacro:if value="${moveit_collision_housing}">
+                <collision>
+                    <origin xyz="0 0 0" rpy="0 0 0"/>
+                    <geometry>
+                        <box size="0.020 0.060 0.020"/>
+                    </geometry>
+                </collision>
+            </xacro:if>
             <inertial>
                 <origin xyz="0 0 0" rpy="0 0 0"/>

File: ur5e_robotiq_description/urdf/ur5e_robotiq.urdf.xacro (robot description, xacro)
@@ -104,4 +104,14 @@
   <xacro:arg name="gripper_model" default="robotiq_linkage"/>
   <xacro:property name="gripper_model" value="$(arg gripper_model)"/>
+  <!-- Stage-3A: planning-only gripper housing collision geometry for
+       gripper_model:=parallel_jaw. Default false reproduces the exact
+       existing (validated) physical model byte-for-byte — Gazebo/simulation
+       launches must never set this true. Only move_group's own independent
+       robot_description build sets it true, so MoveIt's collision-aware
+       planning sees a conservative gripper_base_link housing box while
+       Gazebo's physics stays completely unchanged. See the Stage-3A design
+       audit (2026-09-06) for the geometry derivation and why jaw_fixed_link/
+       jaw_moving_link deliberately receive no collision geometry here. -->
+  <xacro:arg name="moveit_collision_housing" default="false"/>
   <!-- Simulation-only arm spawn state.  The sim launch derives these six
        arguments from scene.yaml milestones.m1.goal_positions.  Defaults keep
@@ -218,5 +228,6 @@
       use_fake_hardware="false"
       fake_sensor_commands="false"
-      include_ros2_control="true">
+      include_ros2_control="true"
+      moveit_collision_housing="$(arg moveit_collision_housing)">
       <origin xyz="0 0 0" rpy="0 0 0"/>
     </xacro:parallel_jaw_gripper>
